Commit message: no se pudo usar moveit2 en ros2 humble, al menos no desde 0 pero si se pueden agregar poses por medio del archivo phantom_ws/src/phantomx_pincher_moveit_config/srdf/phantomx_pincher.xacro

File: phantom_ws/src/phantomx_pincher_moveit_config/srdf/phantomx_pincher.xacro (robot description, xacro)
@@ -50,4 +50,10 @@
       <joint name="${prefix}arm_wrist_flex_joint" value="${pi/2}" />
     </group_state>
+      <group_state group="arm" name="overRightNearCan">
+      <joint name="${prefix}arm_shoulder_pan_joint" value="-${90 * (pi/180)}" />
+      <joint name="${prefix}arm_shoulder_lift_joint" value="${21 * (pi/180)}" />
+      <joint name="${prefix}arm_elbow_flex_joint" value="${80 * (pi/180)}" />
+      <joint name="${prefix}arm_wrist_flex_joint" value="${80 * (pi/180)}" />
+    </group_state>
     <group_state group="gripper" name="open">
       <joint name="${prefix}gripper_finger1_joint" value="0.0158" />
@@ -546,4 +552,98 @@
       reason="Adjacent" />
     -->
+        <!-- ===================================================== -->
+    <!--  KIT PLATFORM COLLISION DISABLES (from kit.xacro)     -->
+    <!--  - Self-collisions between all kit links              -->
+    <!--  - Collisions between arm base and kit links          -->
+    <!-- ===================================================== -->
+    <!--
+      Kit links from kit.xacro:
+        baseFija_link
+        caseBaseRobot_link
+        zonaRecoleccion_link
+        airpump_link
+        manijaTrasera_link
+        manijaDelantera_link
+        canecaLateralIzquierda_link
+        canecaLateralDerecha_link
+        canecaFrontalDerecha_link
+        canecaFrontalIzquierda_link
+    -->
+    <!-- ============================== -->
+    <!-- A) KIT SELF-COLLISIONS (OFF)  -->
+    <!-- ============================== -->
+    <!-- baseFija_link vs others -->
+    <disable_collisions link1="baseFija_link" link2="caseBaseRobot_link"          reason="Never"/>
+    <disable_collisions link1="baseFija_link" link2="zonaRecoleccion_link"        reason="Never"/>
+    <disable_collisions link1="baseFija_link" link2="airpump_link"                reason="Never"/>
+    <disable_collisions link1="baseFija_link" link2="manijaTrasera_link"          reason="Never"/>
+    <disable_collisions link1="baseFija_link" link2="manijaDelantera_link"        reason="Never"/>
+    <disable_collisions link1="baseFija_link" link2="canecaLateralIzquierda_link" reason="Never"/>
+    <disable_collisions link1="baseFija_link" link2="canecaLateralDerecha_link"   reason="Never"/>
+    <disable_collisions link1="baseFija_link" link2="canecaFrontalDerecha_link"   reason="Never"/>
+    <disable_collisions link1="baseFija_link" link2="canecaFrontalIzquierda_link" reason="Never"/>
+    <!-- caseBaseRobot_link vs others -->
+    <disable_collisions link1="caseBaseRobot_link" link2="zonaRecoleccion_link"        reason="Never"/>
+    <disable_collisions link1="caseBaseRobot_link" link2="airpump_link"                reason="Never"/>
+    <disable_collisions link1="caseBaseRobot_link" link2="manijaTrasera_link"          reason="Never"/>
+    <disable_collisions link1="caseBaseRobot_link" link2="manijaDelantera_link"        reason="Never"/>
+    <disable_collisions link1="caseBaseRobot_link" link2="canecaLateralIzquierda_link" reason="Never"/>
+    <disable_collisions link1="caseBaseRobot_link" link2="canecaLateralDerecha_link"   reason="Never"/>
+    <disable_collisions link1="caseBaseRobot_link" link2="canecaFrontalDerecha_link"   reason="Never"/>
+    <disable_collisions link1="caseBaseRobot_link" link2="canecaFrontalIzquierda_link" reason="Never"/>
+    <!-- zonaRecoleccion_link vs others -->
+    <disable_collisions link1="zonaRecoleccion_link" link2="airpump_link"                reason="Never"/>
+    <disable_collisions link1="zonaRecoleccion_link" link2="manijaTrasera_link"          reason="Never"/>
+    <disable_collisions link1="zonaRecoleccion_link" link2="manijaDelantera_link"        reason="Never"/>
+    <disable_collisions link1="zonaRecoleccion_link" link2="canecaLateralIzquierda_link" reason="Never"/>
+    <disable_collisions link1="zonaRecoleccion_link" link2="canecaLateralDerecha_link"   reason="Never"/>
+    <disable_collisions link1="zonaRecoleccion_link" link2="canecaFrontalDerecha_link"   reason="Never"/>
+    <disable_collisions link1="zonaRecoleccion_link" link2="canecaFrontalIzquierda_link" reason="Never"/>
+    <!-- airpump_link vs others -->
+    <disable_collisions link1="airpump_link" link2="manijaTrasera_link"          reason="Never"/>
+    <disable_collisions link1="airpump_link" link2="manijaDelantera_link"        reason="Never"/>
+    <disable_collisions link1="airpump_link" link2="canecaLateralIzquierda_link" reason="Never"/>
+    <disable_collisions link1="airpump_link" link2="canecaLateralDerecha_link"   reason="Never"/>
+    <disable_collisions link1="airpump_link" link2="canecaFrontalDerecha_link"   reason="Never"/>
+    <disable_collisions link1="airpump_link" link2="canecaFrontalIzquierda_link" reason="Never"/>
+    <!-- manijaTrasera_link vs others -->
+    <disable_collisions link1="manijaTrasera_link" link2="manijaDelantera_link"        reason="Never"/>
+    <disable_collisions link1="manijaTrasera_link" link2="canecaLateralIzquierda_link" reason="Never"/>
+    <disable_collisions link1="manijaTrasera_link" link2="canecaLateralDerecha_link"   reason="Never"/>
+    <disable_collisions link1="manijaTrasera_link" link2="canecaFrontalDerecha_link"   reason="Never"/>
+    <disable_collisions link1="manijaTrasera_link" link2="canecaFrontalIzquierda_link" reason="Never"/>
+    <!-- manijaDelantera_link vs others -->
+    <disable_collisions link1="manijaDelantera_link" link2="canecaLateralIzquierda_link" reason="Never"/>
+    <disable_collisions link1="manijaDelantera_link" link2="canecaLateralDerecha_link"   reason="Never"/>
+    <disable_collisions link1="manijaDelantera_link" link2="canecaFrontalDerecha_link"   reason="Never"/>
+    <disable_collisions link1="manijaDelantera_link" link2="canecaFrontalIzquierda_link" reason="Never"/>
+    <!-- canecaLateralIzquierda_link vs others -->
+    <disable_collisions link1="canecaLateralIzquierda_link" link2="canecaLateralDerecha_link"   reason="Never"/>
+    <disable_collisions link1="canecaLateralIzquierda_link" link2="canecaFrontalDerecha_link"   reason="Never"/>
+    <disable_collisions link1="canecaLateralIzquierda_link" link2="canecaFrontalIzquierda_link" reason="Never"/>
+    <!-- canecaLateralDerecha_link vs others -->
+    <disable_collisions link1="canecaLateralDerecha_link" link2="canecaFrontalDerecha_link"   reason="Never"/>
+    <disable_collisions link1="canecaLateralDerecha_link" link2="canecaFrontalIzquierda_link" reason="Never"/>
+    <!-- canecaFrontalDerecha_link vs others -->
+    <disable_collisions link1="canecaFrontalDerecha_link" link2="canecaFrontalIzquierda_link" reason="Never"/>
+    <!-- ================================================= -->
+    <!-- B) ARM BASE vs KIT COLLISIONS (OFF)              -->
+    <!--    Arm base link assumed to be ${prefix}arm_base_link -->
+    <!-- ================================================= -->
+    <disable_collisions link1="${prefix}arm_base_link" link2="baseFija_link"               reason="Never"/>
+    <disable_collisions link1="${prefix}arm_base_link" link2="caseBaseRobot_link"         reason="Never"/>
+    <disable_collisions link1="${prefix}arm_base_link" link2="zonaRecoleccion_link"       reason="Never"/>
+    <disable_collisions link1="${prefix}arm_base_link" link2="airpump_link"               reason="Never"/>
+    <disable_collisions link1="${prefix}arm_base_link" link2="manijaTrasera_link"         reason="Never"/>
+    <disable_collisions link1="${prefix}arm_base_link" link2="manijaDelantera_link"       reason="Never"/>
+    <disable_collisions link1="${prefix}arm_base_link" link2="canecaLateralIzquierda_link" reason="Never"/>
+    <disable_collisions link1="${prefix}arm_base_link" link2="canecaLateralDerecha_link"  reason="Never"/>
+    <disable_collisions link1="${prefix}arm_base_link" link2="canecaFrontalDerecha_link"  reason="Never"/>
+    <disable_collisions link1="${prefix}arm_base_link" link2="canecaFrontalIzquierda_link" reason="Never"/>
+    <!-- Disable collision between shoulder pan servo and case base on the kit -->
+    <disable_collisions
+        link1="${prefix}arm_shoulder_pan_servo_link"
+        link2="caseBaseRobot_link"
+        reason="Never"/>
   </xacro:macro>
 </robot>
