Commit message: El gripper se cambio a movimiento prismatico, ahora se puede hacer el movimiento del gripper del robot en Rviz de open a closed

File: phantom_ws/src/phantomx_pincher_description/urdf/phantomx_pincher.urdf (robot description, URDF)
Before this commit: robot phantomx_pincher, 35 links, 34 joints
Joints:
- joint phantomx_pincher_gripper_finger1_joint: limit lower=0.001 upper=0.0158 effort=30 velocity=0.01 -> lower=0.00375 upper=0.01955 effort=30 velocity=0.01
- joint phantomx_pincher_gripper_finger2_joint: limit lower=0.001 upper=0.0158 effort=30 velocity=0.01 -> lower=0.00375 upper=0.01955 effort=30 velocity=0.01
