Commit message: Se añadio la visualizacion y colision de la ventosa, se modifico el archivo phantomx_pincher_arm.xacro en el paquete phantomx_pincher_description y tambien se modificaron los archivos dentro de la carpeta srdf del paquete phantomx_pincher_moveit_config

File: phantom_ws/src/phantomx_pincher_description/urdf/phantomx_pincher_arm.xacro (robot description, xacro)
@@ -329,5 +329,4 @@
           gazebo_preserve_fixed_joint="${gazebo_preserve_fixed_joint}"/>
     </xacro:unless>
-    <!-- SUCTION CUP-->
     <!-- Adaptador de ventosa montado en el efector final -->
     <link name="${prefix}coupling_tool_end_effector_link">
@@ -338,5 +337,5 @@
                 scale="0.001 0.001 0.001" />
             </geometry>
-            <material name="gray" />
+            <material name="blue" />
         </visual>
         <collision>
@@ -361,5 +360,36 @@
         <origin xyz="0.000008282 0 -0.038" rpy="${PI/2} 0 ${PI/2}"/>
     </joint>
-    <!-- ==================== -->
+    <!-- suction cup link and joint-->
+    <link name="${prefix}suction_cup_link">
+        <visual>
+            <origin xyz="0 0 0" rpy="0 0 0"/>
+            <geometry>
+                <mesh filename="package://phantomx_pincher_description/meshes/DAE/suctionCupGripper.dae"
+                scale="0.001 0.001 0.001" />
+            </geometry>
+            <material name="blue" />
+        </visual>
+        <collision>
+            <origin xyz="-0.0585 0.010 -0.024" rpy="${PI/2} 0 0"/>
+            <geometry>
+                <mesh filename="package://phantomx_pincher_description/meshes/STL/suctionCupGripper.stl"
+                scale="0.001 0.001 0.001" />
+            </geometry>
+        </collision>
+        <inertial>
+            <origin xyz="-0.077757 -0.027995 0.000" rpy="0 0 0"/>
+            <mass value="0.025"/> <!-- kg -->
+            <inertia
+                ixx="0.000005868"  ixy="-0.000007410"  ixz="0.000000000"
+                                iyy="0.000021405"   iyz="0.000000000"
+                                                    izz="0.000026615"/>
+        </inertial><!-- kg *  m^2 -->
+    </link>
+    <joint name="${prefix}suction_cup_joint" type="fixed">
+        <parent link="${prefix}coupling_tool_end_effector_link"/>
+        <child link="${prefix}suction_cup_link"/>
+        <origin xyz="0 -0.01075 0.049" rpy="0 0 -${PI/2}"/>
+    </joint>
+    <!-- ====================  ${0.0115 / 2}-->
     <!-- Efector final        -->
     <!-- ==================== -->

File: phantom_ws/src/phantomx_pincher_moveit_config/srdf/phantomx_pincher.xacro (robot description, xacro)
@@ -693,6 +693,48 @@
       <disable_collisions link1="${prefix}coupling_tool_end_effector_link"
         link2="${prefix}arm_shoulder_F3_0_link" reason="Never" />
+<!-- ============================== -->
+      <!-- C) Suction Cup SELF COLLISIONS OFF   -->
+      <!-- ============================== -->
+      <!-- suction_cup_link collisions -->
+      <disable_collisions link1="${prefix}suction_cup_link"
+        link2="${prefix}coupling_tool_end_effector_link" reason="Adjacent" />
+      <disable_collisions link1="${prefix}suction_cup_link"
+        link2="${prefix}end_effector" reason="Adjacent" />
+      <disable_collisions link1="${prefix}suction_cup_link"
+        link2="${prefix}gripper_finger_base_link" reason="Never" />
+      <disable_collisions link1="${prefix}suction_cup_link"
+        link2="${prefix}gripper_finger1_link" reason="Never" />
+      <disable_collisions link1="${prefix}suction_cup_link"
+        link2="${prefix}gripper_finger2_link" reason="Never" />
+      <disable_collisions link1="${prefix}suction_cup_link"
+        link2="${prefix}gripper_servo_link" reason="Never" />
+      <disable_collisions link1="${prefix}suction_cup_link"
+        link2="${prefix}arm_wrist_flex_servo_link" reason="Never" />
+      <disable_collisions link1="${prefix}suction_cup_link"
+        link2="${prefix}arm_wrist_flex_link" reason="Never" />
+      <disable_collisions link1="${prefix}suction_cup_link"
+        link2="${prefix}arm_wrist_F3_0_link" reason="Never" />
+      <disable_collisions link1="${prefix}suction_cup_link"
+        link2="${prefix}arm_elbow_flex_servo_link" reason="Never" />
+      <disable_collisions link1="${prefix}suction_cup_link"
+        link2="${prefix}arm_elbow_flex_link" reason="Never" />
+      <disable_collisions link1="${prefix}suction_cup_link"
+        link2="${prefix}arm_elbow_F3_0_link" reason="Never" />
+      <disable_collisions link1="${prefix}suction_cup_link"
+        link2="${prefix}arm_elbow_F10_0_link" reason="Never" />
+      <disable_collisions link1="${prefix}suction_cup_link"
+        link2="${prefix}arm_elbow_F10_1_link" reason="Never" />
+      <disable_collisions link1="${prefix}suction_cup_link"
+        link2="${prefix}arm_elbow_F10_2_link" reason="Never" />
+      <disable_collisions link1="${prefix}suction_cup_link"
+        link2="${prefix}arm_shoulder_F10_0_link" reason="Never" />
+      <disable_collisions link1="${prefix}suction_cup_link"
+        link2="${prefix}arm_shoulder_F10_1_link" reason="Never" />
+      <disable_collisions link1="${prefix}suction_cup_link"
+        link2="${prefix}arm_shoulder_F10_2_link" reason="Never" />
+      <disable_collisions link1="${prefix}suction_cup_link"
+        link2="${prefix}arm_shoulder_F3_0_link" reason="Never" />
     <!-- ================================================= -->
-    <!-- C) ARM BASE vs KIT COLLISIONS (OFF)              -->
+    <!-- D) ARM BASE vs KIT COLLISIONS (OFF)              -->
     <!--    Arm base link assumed to be ${prefix}arm_base_link -->
     <!-- ================================================= -->
