Commit message: Se añadieron varios archivos .DAE en phantomx_pinhcer_description en meshes en DAE, estos archivos se usaron para modificar el archivo kit.xacro en la carpeta urdf dentro del paquete phantomx_pincher_description en urdf. Esto mejora el aspecto visual de la visualizacion. Aun falta añadir varios y reemplazar el archivo visual de las canecas.

File: phantom_ws/src/phantomx_pincher_description/urdf/kit.xacro (robot description, xacro)
@@ -26,7 +26,66 @@
   <link name="baseFija_link">
     <visual>
-      <origin xyz="0.155 0 0.000" rpy="0 0 -${PI/2}" />
-      <geometry>
-        <mesh filename="package://phantomx_pincher_description/meshes/STL/baseElementosFijos.stl"
+      <origin xyz="0 0 0.009" rpy="-${PI/2} 0 -${PI/2}" />
+      <geometry>
+        <mesh filename="package://phantomx_pincher_description/meshes/DAE/ensambleBase.dae"
+              scale="0.001 0.001 0.001" />
+      </geometry>
+      <material name="gray" />
+    </visual>
+    <collision> <!-- base -->
+      <origin xyz="0.155 0.0 0.0045" rpy="0 0 -${PI/2}" />
+      <geometry>
+        <box size="0.360 0.554 0.009" />
+      	<material name="gray" />
+      </geometry>
+    </collision>
+    <collision>
+      <origin xyz="-0.112 0 0.03425" rpy="-${PI/2} 0 ${PI/2}" />
+      <geometry> <!--manijaTrasera-->
+        <box size="0.136 0.0505 0.020" />
+      	<material name="gray" />
+      </geometry>
+    </collision>
+    <collision>
+      <origin xyz="0.422 0 0.03425" rpy="-${PI/2} 0 ${PI/2}" />
+      <geometry> <!-- manijaDelantera -->
+        <box size="0.136 0.0505 0.020" />
+      	<material name="gray" />
+      </geometry>
+    </collision>
+    <collision>
+      <origin xyz="0.418 0.143625 0.024" rpy="0 0 0" />
+      <geometry> <!-- pata Delantera izquierda -->
+        <box size="0.028 0.05175 0.030" />
+      	<material name="gray" />
+      </geometry>
+    </collision>
+    <collision>
+      <origin xyz="0.418 -0.143625 0.024" rpy="0 0 0" />
+      <geometry> <!-- pata Delantera derecha -->
+        <box size="0.028 0.05175 0.030" />
+      	<material name="gray" />
+      </geometry>
+    </collision>
+    <collision>
+      <origin xyz="-0.112 0.143625 0.024" rpy="0 0 0" />
+      <geometry> <!-- pata trasera izquierda -->
+        <box size="0.028 0.05175 0.030" />
+      	<material name="gray" />
+      </geometry>
+    </collision>
+    <collision>
+      <origin xyz="-0.112 -0.143625 0.024" rpy="0 0 0" />
+      <geometry> <!-- pata trasera derecha -->
+        <box size="0.028 0.05175 0.030" />
+      	<material name="gray" />
+      </geometry>
+    </collision>
+  </link>
+  <link name="caseBaseRobot_link">
+    <visual>
+      <origin xyz="0.0 0.0 0.0" rpy="${PI/2} 0 ${PI/2}" />
+      <geometry>
+        <mesh filename="package://phantomx_pincher_description/meshes/DAE/ensambleBaseBrazo.dae"
               scale="0.001 0.001 0.001" />
       </geometry>
@@ -34,26 +93,9 @@
     </visual>
     <collision>
-      <origin xyz="0.155 0 0.0045" rpy="0 0 -${PI/2}" />
-      <geometry>
-        <box size="0.360 0.554 0.009" />
-      </geometry>
-      <material name="black" />
-    </collision>
-  </link>
-  <link name="caseBaseRobot_link">
-    <visual>
-      <origin xyz="0 0 0" rpy="${PI} 0 ${PI/2}" />
-      <geometry>
-        <mesh filename="package://phantomx_pincher_description/meshes/STL/caseBaseRobot.stl"
-              scale="0.001 0.001 0.001" />
-      </geometry>
-      <material name="gray" />
-    </visual>
-    <collision>
-        <origin xyz="0 0 -0.024" rpy="${PI} 0 ${PI/2}" />
+        <origin xyz="-0.01325 0.0 -${0.024 - 0.005}" rpy="${PI} 0 ${PI/2}" />
         <geometry>
             <box size="0.066 0.074 0.048" />
         </geometry>
-        <material name="gray" />
+        <material name="black" />
     </collision>
   </link>
@@ -61,5 +103,5 @@
     <parent link="baseFija_link" />
     <child link="caseBaseRobot_link" />
-    <origin xyz="-0.01325 0 0.054" rpy="0 0 0" />
+    <origin xyz="0.0 0.0 ${0.048+0.004}" rpy="0 0 0" />
   </joint>
   <link name="zonaRecoleccion_link">
@@ -87,17 +129,17 @@
   <link name="airpump_link">
     <visual>
-      <origin xyz="0 0 0" rpy="${PI/2} 0 -${PI/2}" />
-      <geometry>
-        <mesh filename="package://phantomx_pincher_description/meshes/STL/ensambleAirpump.stl"
-              scale="0.001 0.001 0.001" />
-      </geometry>
-      <material name="gray" />
-    </visual>
-    <collision>
-      <origin xyz="-0.0647 0 0.014" rpy="${PI/2} 0 -${PI/2}" />
+      <origin xyz="0 0 0" rpy="0 0 -${PI/2}" />
+      <geometry>
+        <mesh filename="package://phantomx_pincher_description/meshes/DAE/ensambleAirpump.dae"
+              scale="0.001 0.001 0.001" />
+      </geometry>
+      <material name="black" />
+    </visual>
+    <collision>
+      <origin xyz="-0.0647 0.0 0.014" rpy="${PI/2} 0 -${PI/2}" />
       <geometry>
         <box size="0.062 0.0405 0.067" />
       </geometry>
-      <material name="gray" />
+      <material name="black" />
     </collision>
   </link>
@@ -106,48 +148,4 @@
     <child link="airpump_link" />
     <origin xyz="0 0 0.009" rpy="0 0 0" />
-  </joint>
-  <link name="manijaTrasera_link">
-    <visual>
-      <origin xyz="0 0 0" rpy="-${PI/2} 0 ${PI/2}" />
-      <geometry>
-        <mesh filename="package://phantomx_pincher_description/meshes/STL/manija.stl"
-              scale="0.001 0.001 0.001" />
-      </geometry>
-      <material name="gray" />
-    </visual>
-    <collision>
-      <origin xyz="-0.010 0 0" rpy="-${PI/2} 0 ${PI/2}" />
-      <geometry>
-        <box size="0.136 0.0505 0.020" />
-      </geometry>
-      <material name="gray" />
-    </collision>
-  </link>
-  <joint name="base_manijaTrasera_joint" type="fixed">
-    <parent link="baseFija_link" />
-    <child link="manijaTrasera_link" />
-    <origin xyz="-0.102 0 0.03425" rpy="0 0 0" />
-  </joint>
-  <link name="manijaDelantera_link">
-    <visual>
-      <origin xyz="0 0 0" rpy="-${PI/2} 0 ${PI/2}" />
-      <geometry>
-        <mesh filename="package://phantomx_pincher_description/meshes/STL/manija.stl"
-              scale="0.001 0.001 0.001" />
-      </geometry>
-      <material name="gray" />
-    </visual>
-    <collision>
-      <origin xyz="-0.010 0 0" rpy="-${PI/2} 0 ${PI/2}" />
-      <geometry>
-        <box size="0.136 0.0505 0.020" />
-      </geometry>
-      <material name="gray" />
-    </collision>
-  </link>
-  <joint name="base_manijaDelantera_joint" type="fixed">
-    <parent link="baseFija_link" />
-    <child link="manijaDelantera_link" />
-    <origin xyz="0.432 0 0.03425" rpy="0 0 0" />
   </joint>
   <link name="canecaLateralIzquierda_link">
@@ -259,4 +257,6 @@
 Lateral derecha	0 0 -${PI/2}
 Lateral izquierda	0 0 ${PI/2}
+sudo apt install ros-jazzy-urdf-tutorial
+ros2 launch urdf_tutorial display.launch.py model:=/home/unpi/ros2/KIT_Phantom_X_Pincher_ROS2/phantom_ws/src/phantomx_pincher_description/urdf/kit.xacro
   -->
 </robot>

Commit message: phantomx_pincher_description: add caneca DAE meshes and update kit.xacro
Added DAE mesh files:
- meshes/DAE/canecaAmarilla.dae
- meshes/DAE/canecaAzul.dae
- meshes/DAE/canecaRojo.dae
- meshes/DAE/canecaVerde.dae
- meshes/STL/canastilla.stl

Modified:
- urdf/kit.xacro: added visual and collision tags referencing the new
  caneca DAE files so they render correctly in RViz

File: phantom_ws/src/phantomx_pincher_description/urdf/kit.xacro (robot description, xacro)
@@ -21,4 +21,5 @@
   <material name="blue"><color rgba="0 0 1 1"/></material>
   <material name="purple"><color rgba="0.5 0 0.5 1"/></material>
+  <material name="orange"><color rgba="1.0 0.5 0.0 1"/></material>
   <!-- ============================= -->
   <!-- 🧱 Robot Geometry -->
@@ -37,5 +38,4 @@
       <geometry>
         <box size="0.360 0.554 0.009" />
-      	<material name="gray" />
       </geometry>
     </collision>
@@ -44,5 +44,4 @@
       <geometry> <!--manijaTrasera-->
         <box size="0.136 0.0505 0.020" />
-      	<material name="gray" />
       </geometry>
     </collision>
@@ -51,5 +50,4 @@
       <geometry> <!-- manijaDelantera -->
         <box size="0.136 0.0505 0.020" />
-      	<material name="gray" />
       </geometry>
     </collision>
@@ -58,5 +56,4 @@
       <geometry> <!-- pata Delantera izquierda -->
         <box size="0.028 0.05175 0.030" />
-      	<material name="gray" />
       </geometry>
     </collision>
@@ -65,22 +62,55 @@
       <geometry> <!-- pata Delantera derecha -->
         <box size="0.028 0.05175 0.030" />
-      	<material name="gray" />
-      </geometry>
-    </collision>
-    <collision>
-      <origin xyz="-0.112 0.143625 0.024" rpy="0 0 0" />
+      </geometry>
+    </collision>
+    <collision>
+      <origin xyz="-${0.112 - 0.004} 0.143625 0.024" rpy="0 0 0" />
       <geometry> <!-- pata trasera izquierda -->
         <box size="0.028 0.05175 0.030" />
-      	<material name="gray" />
-      </geometry>
-    </collision>
-    <collision>
-      <origin xyz="-0.112 -0.143625 0.024" rpy="0 0 0" />
+      </geometry>
+    </collision>
+    <collision>
+      <origin xyz="-${0.112 - 0.004} -0.143625 0.024" rpy="0 0 0" />
       <geometry> <!-- pata trasera derecha -->
         <box size="0.028 0.05175 0.030" />
-      	<material name="gray" />
-      </geometry>
-    </collision>
-  </link>
+      </geometry>
+    </collision>
+  </link>
+  <link name="soporteCamara_link">
+    <visual>
+      <origin xyz="0.0 0.0 0.0" rpy="-${PI/2} 0 -${PI/2}" />
+      <geometry>
+        <mesh filename="package://phantomx_pincher_description/meshes/DAE/ensambleSoporteC270Webcam.dae"
+              scale="0.001 0.001 0.001" />
+      </geometry>
+      <material name="purple" />
+    </visual>
+    <collision> <!-- mastil -->
+        <origin xyz="0.0 0.0 ${0.353 - 0.005}" rpy="0 0 0" />
+        <geometry>
+            <box size="0.040 0.062 0.706" />
+        </geometry>
+        <material name="purple" />
+    </collision>
+    <collision> <!-- acople Camara -->
+        <origin xyz="-${0.088 - 0.02} 0.0 ${0.706 - 0.02}" rpy="0 0 0" />
+        <geometry>
+            <box size="0.176 0.062 0.04" />
+        </geometry>
+        <material name="purple" />
+    </collision>
+    <collision> <!-- Camara -->
+        <origin xyz="-${0.176 - 0.030} -0.0165 ${0.706 - 0.038}" rpy="0 0 0" />
+        <geometry>
+            <box size="0.040 0.072 0.076" />
+        </geometry>
+        <material name="purple" />
+    </collision>
+  </link>
+  <joint name="base_soporteCamara_joint" type="fixed">
+    <parent link="baseFija_link" />
+    <child link="soporteCamara_link" />
+    <origin xyz="0.26025 0.0 ${0.005 + 0.009}" rpy="0 0 0" />
+  </joint>
   <link name="caseBaseRobot_link">
     <visual>
@@ -92,8 +122,15 @@
       <material name="black" />
     </visual>
-    <collision>
+    <collision> <!-- base brazo -->
         <origin xyz="-0.01325 0.0 -${0.024 - 0.005}" rpy="${PI} 0 ${PI/2}" />
         <geometry>
             <box size="0.066 0.074 0.048" />
+        </geometry>
+        <material name="black" />(0.048-0.03258)
+    </collision>
+    <collision> <!-- Placa numero -->
+        <origin xyz="0.020 0.0 -0.010" rpy="0 -${PI * (17/180)} 0" />
+        <geometry>
+            <box size="0.005 0.022 0.030" />
         </geometry>
         <material name="black" />
@@ -136,10 +173,15 @@
       <material name="black" />
     </visual>
-    <collision>
+    <collision> <!-- carcasa arimpump -->
       <origin xyz="-0.0647 0.0 0.014" rpy="${PI/2} 0 -${PI/2}" />
       <geometry>
         <box size="0.062 0.0405 0.067" />
       </geometry>
-      <material name="black" />
+    </collision>
+    <collision> <!-- Placa numero -->
+        <origin xyz="-0.0747 0.0 ${0.0325}" rpy="0 0 0" />
+        <geometry>
+            <box size="0.030 0.022 0.005" />
+        </geometry>
     </collision>
   </link>
@@ -151,4 +193,12 @@
   <link name="canecaLateralIzquierda_link">
     <visual>
+      <origin xyz="0 0 0.003" rpy="-${PI/2} 0 -${PI/2}" />
+      <geometry>
+        <mesh filename="package://phantomx_pincher_description/meshes/DAE/canecaRojo.dae"
+              scale="0.001 0.001 0.001" />
+      </geometry>
+      <material name="red" />
+    </visual>
+    <collision>
       <origin xyz="0 0 0" rpy="0 0 -${PI/2}" />
       <geometry>
@@ -156,13 +206,4 @@
               scale="0.001 0.001 0.001" />
       </geometry>
-      <material name="red" />
-    </visual>
-    <collision>
-      <origin xyz="0 0 0" rpy="0 0 -${PI/2}" />
-      <geometry>
-        <mesh filename="package://phantomx_pincher_description/meshes/STL/canecaGrande.stl"
-              scale="0.001 0.001 0.001" />
-      </geometry>
-      <material name="red" />
     </collision>
   </link>
@@ -174,4 +215,12 @@
   <link name="canecaLateralDerecha_link">
     <visual>
+      <origin xyz="0 0 0.003" rpy="-${PI/2} 0 ${PI/2}" />
+      <geometry>
+        <mesh filename="package://phantomx_pincher_description/meshes/DAE/canecaAmarilla.dae"
+              scale="0.001 0.001 0.001" />
+      </geometry>
+      <material name="yellow" />
+    </visual>
+    <collision>
       <origin xyz="0 0 0" rpy="0 0 ${PI/2}" />
       <geometry>
@@ -179,13 +228,4 @@
               scale="0.001 0.001 0.001" />
       </geometry>
-      <material name="yellow" />
-    </visual>
-    <collision>
-      <origin xyz="0 0 0" rpy="0 0 ${PI/2}" />
-      <geometry>
-        <mesh filename="package://phantomx_pincher_description/meshes/STL/canecaGrande.stl"
-              scale="0.001 0.001 0.001" />
-      </geometry>
-      <material name="yellow" />
     </collision>
   </link>
@@ -197,4 +237,12 @@
   <link name="canecaFrontalDerecha_link">
     <visual>
+      <origin xyz="0 0 0.003" rpy="-${PI/2} 0 ${PI*((180-25.5)/180)}" />
+      <geometry>
+        <mesh filename="package://phantomx_pincher_description/meshes/DAE/canecaAzul.dae"
+              scale="0.001 0.001 0.001" />
+      </geometry>
+      <material name="blue" />
+    </visual>
+    <collision>
       <origin xyz="0 0 0" rpy="0 0 ${PI*((180-25.5)/180)}" />
       <geometry>
@@ -202,13 +250,4 @@
               scale="0.001 0.001 0.001" />
       </geometry>
-      <material name="green" />
-    </visual>
-    <collision>
-      <origin xyz="0 0 0" rpy="0 0 ${PI*((180-25.5)/180)}" />
-      <geometry>
-        <mesh filename="package://phantomx_pincher_description/meshes/STL/canecaGrande.stl"
-              scale="0.001 0.001 0.001" />
-      </geometry>
-      <material name="green" />
     </collision>
   </link>
@@ -218,6 +257,14 @@
     <origin xyz="0.19397558339 -0.09252160722 0.016" rpy="0 0 0" />
   </joint>
-  <link name="canecaFrontalIzquierda_link">
-    <visual>
+  <link name="canecaFrontalIzquierda_link"> <!-- caneca azul -0.05 -0.074 0.003 0.20724702645 0.18083847310-->
+    <visual>
+      <origin xyz="0 0 0.003" rpy="-${PI/2} 0 ${PI*(25.5/180) + PI}" />
+      <geometry>
+        <mesh filename="package://phantomx_pincher_description/meshes/DAE/canecaVerde.dae"
+              scale="0.001 0.001 0.001" />
+      </geometry>
+      <material name="green" />
+    </visual>
+    <collision>
       <origin xyz="0 0 0" rpy="0 0 ${PI*(25.5/180) + PI}" />
       <geometry>
@@ -225,13 +272,4 @@
               scale="0.001 0.001 0.001" />
       </geometry>
-      <material name="blue" />
-    </visual>
-    <collision>
-      <origin xyz="0 0 0" rpy="0 0 ${PI*(25.5/180) + PI}" />
-      <geometry>
-        <mesh filename="package://phantomx_pincher_description/meshes/STL/canecaGrande.stl"
-              scale="0.001 0.001 0.001" />
-      </geometry>
-      <material name="blue" />
     </collision>
   </link>
@@ -240,4 +278,116 @@
     <child link="canecaFrontalIzquierda_link" />
     <origin xyz="0.19397558339 0.09252160722 0.016" rpy="0 0 0" />
+  </joint>
+  <link name="raspberry_link">
+    <visual>
+      <origin xyz="0 0 0" rpy="-${PI/2} 0 ${PI}" />
+      <geometry>
+        <mesh filename="package://phantomx_pincher_description/meshes/DAE/ensambleRaspberrypi.dae"
+              scale="0.001 0.001 0.001" />
+      </geometry>
+      <material name="orange" />
+    </visual>
+    <collision>
+      <origin xyz="0 0 0" rpy="0 0 0" />
+      <geometry>
+        <box size="0.134 0.075 0.068" />
+      </geometry>
+    </collision>
+  </link>
+  <joint name="base_raspberry_joint" type="fixed">
+    <parent link="baseFija_link" />
+    <child link="raspberry_link" />
+    <origin xyz="0.330 0.1425 ${0.0345 + 0.009}" rpy="0 0 0" />
+  </joint>
+  <link name="canastilla_link">
+    <visual>
+      <origin xyz="0 0 0" rpy="0 0 0" />
+      <geometry>
+        <mesh filename="package://phantomx_pincher_description/meshes/STL/canastilla.stl"
+              scale="0.001 0.001 0.001" />
+      </geometry>
+      <material name="blue" />
+    </visual>
+    <collision><!-- pared larga izquierda-->
+      <origin xyz="0 0.1915 ${0.190 / 2}" rpy="0 0 0" />
+      <geometry>
+        <box size="0.600 0.017 0.190" />
+      </geometry>
+    </collision>
+    <collision><!-- pared larga derecha-->
+      <origin xyz="0 -0.1915 ${0.190 / 2}" rpy="0 0 0" />
+      <geometry>
+        <box size="0.600 0.017 0.190" />
+      </geometry>
+    </collision>
+    <collision><!-- pared corta delantera-->
+      <origin xyz="0.2915 0.0 ${0.190 / 2}" rpy="0 0 0" />
+      <geometry>
+        <box size="0.017 0.366 0.190" />
+      </geometry>
+    </collision>
+    <collision><!-- pared corta trasera-->
+      <origin xyz="-0.2915 0.0 ${0.190 / 2}" rpy="0 0 0" />
+      <geometry>
+        <box size="0.017 0.366 0.190" />
+      </geometry>
+    </collision>
+    <collision><!-- esquina rotada trasera izquierda -->
+      <origin xyz="-0.283 0.183 ${0.190 / 2}" rpy="0 0 ${PI/4}" />
+      <geometry>
+        <box size="0.018 0.018 0.190" />
+      </geometry>
+    </collision>
+    <collision><!-- esquina rotada trasera derecha -->
+      <origin xyz="-0.283 -0.183 ${0.190 / 2}" rpy="0 0 ${PI/4}" />
+      <geometry>
+        <box size="0.018 0.018 0.190" />
+      </geometry>
+    </collision>
+    <collision><!-- esquina rotada delantera izquierda -->
+      <origin xyz="0.283 0.183 ${0.190 / 2}" rpy="0 0 ${PI/4}" />
+      <geometry>
+        <box size="0.018 0.018 0.190" />
+      </geometry>
+    </collision>
+    <collision><!-- esquina rotada delantera derecha -->
+      <origin xyz="0.283 -0.183 ${0.190 / 2}" rpy="0 0 ${PI/4}" />
+      <geometry>
+        <box size="0.018 0.018 0.190" />
+      </geometry>
+    </collision>
+  </link>
+  <joint name="base_canastilla_joint" type="fixed">
+    <parent link="baseFija_link" />
+    <child link="canastilla_link" />
+    <origin xyz="0.154 0 -${0.011 + 0.0145}" rpy="0 0 0" />
+  </joint>
+  <link name="electronics_link">
+    <visual> <!-- Multitoma-->
+      <origin xyz="0.28225 -0.1515 ${0.0275 + 0.009}" rpy="0 0 ${PI/2}" />
+      <geometry>
+        <mesh filename="package://phantomx_pincher_description/meshes/DAE/ensambleMultitoma.dae"
+              scale="0.001 0.001 0.001" />
+      </geometry>
+      <material name="yellow" />
+    </visual>
+    <visual> <!-- Arbotix -->
+      <origin xyz="0.34796868605 0.11930139262 ${0.04542796419 + 0.009}" rpy="0 0 0" />
+      <geometry>
+        <mesh filename="package://phantomx_pincher_description/meshes/DAE/ensambleArbotix.dae"
+              scale="0.001 0.001 0.001" />
+      </geometry>
+    </visual>
+    <collision> <!-- bloque completo de electronica -->
+      <origin xyz="${0.346 - 0.000125} -0.0375 ${(0.151 / 2) + 0.009}" rpy="0 0 0" />
+      <geometry>
+        <box size="${0.125 + 0.00325+0.0035 } ${0.250 + 0.0245 + 0.0105} 0.151" />
+      </geometry>
+    </collision>
+  </link>
+  <joint name="base_electronics_joint" type="fixed">
+    <parent link="baseFija_link" />
+    <child link="electronics_link" />
+    <origin xyz="0 0 0" rpy="0 0 0" />
   </joint>
   <!-- ============================= -->
@@ -253,10 +403,11 @@
 Superior (normal)	0 0 0
 Inferior (desde abajo)	${PI} 0 0
-Frontal	0 -${PI/2} 0
-Trasera	0 ${PI/2} 0
-Lateral derecha	0 0 -${PI/2}
-Lateral izquierda	0 0 ${PI/2}
+Frontal			0 -${PI/2} 0
+Trasera			0 ${PI/2} 0
+Lateral derecha		-${PI/2} 0 0
+Lateral izquierda	${PI/2} 0 0
 sudo apt install ros-jazzy-urdf-tutorial
 ros2 launch urdf_tutorial display.launch.py model:=/home/unpi/ros2/KIT_Phantom_X_Pincher_ROS2/phantom_ws/src/phantomx_pincher_description/urdf/kit.xacro
+ros2 launch urdf_tutorial display.launch.py model:=/home/unpi/ros2/KIT_Phantom_X_Pincher_ROS2/phantom_ws/src/phantomx_pincher_description/urdf/kit.xacro ; pkill -f rviz2 ; pkill -f robot_state_publisher ; pkill -f joint_state_publisher
   -->
 </robot>
