Commit message: Se han añadido todos los componentes necesarios para el funcionamiento con ventosa, falta quiza buscar una mera de activar o desactivar la ventosa. Tambien se ha definido el TCP de la ventosa. El siguiente paso es desactivar el suction cop para formalizar la version 2 del repositorio y empezar a hacer las guias

File: phantom_ws/src/phantomx_pincher_description/urdf/kit.xacro (robot description, xacro)
@@ -410,4 +410,5 @@
 ros2 launch urdf_tutorial display.launch.py model:=/home/unpi/ros2/KIT_Phantom_X_Pincher_ROS2/phantom_ws/src/phantomx_pincher_description/urdf/kit.xacro
 ros2 launch urdf_tutorial display.launch.py model:=/home/unpi/ros2/KIT_Phantom_X_Pincher_ROS2/phantom_ws/src/phantomx_pincher_description/urdf/kit.xacro ; pkill -f rviz2 ; pkill -f robot_state_publisher ; pkill -f joint_state_publisher
+ros2 launch urdf_tutorial display.launch.py model:=/home/unpi/ros2/KIT_Phantom_X_Pincher_ROS2/phantom_ws/src/phantomx_pincher_description/urdf/phantomx_pincher.urdf.xacro
   -->
 </robot>

File: phantom_ws/src/phantomx_pincher_description/urdf/phantomx_pincher_arm.xacro (robot description, xacro)
@@ -356,7 +356,7 @@
     </link>
     <joint name="${prefix}acople_suction_cup_joint" type="fixed">
-        <parent link="${prefix}end_effector"/>
+        <parent link="${prefix}gripper_servo_link"/>
         <child link="${prefix}coupling_tool_end_effector_link"/>
-        <origin xyz="0.000008282 0 -0.038" rpy="${PI/2} 0 ${PI/2}"/>
+        <origin xyz="0 0 0" rpy="0 ${PI} 0"/>
     </joint>
     <!-- suction cup link and joint-->
@@ -397,4 +397,8 @@
          No tiene geometría; es el punto de referencia que usa MoveIt para
          calcular la cinemática inversa y planificar movimientos. -->
+    <!-- ==================== -->
+    <!-- TCP garra, gripper   -->
+    <!-- ==================== -->
+    <!-- TCP garra, gripper-->
     <xacro:phantomx_pincher_virtual_link
         parent="${prefix}gripper_finger_base_link"
@@ -404,4 +408,16 @@
         gazebo_preserve_fixed_joint="${gazebo_preserve_fixed_joint}"
         />
+    <!-- ==================== -->
+    <!-- TCP ventosa   -->
+    <!-- ==================== -->
+    <!-- TCP suction cop, ventosa
+    <xacro:phantomx_pincher_virtual_link
+        parent="${prefix}suction_cup_link"
+        link_name="${prefix}end_effector"
+        joint_origin_xyz="-0.114 0 -0.029"
+        joint_origin_rpy="${pi/2} ${-pi/2} ${pi/2}"
+        gazebo_preserve_fixed_joint="${gazebo_preserve_fixed_joint}"
+    />
+    -->
     <!-- ==================== -->
     <!-- ROS 2 Control        -->
