Commit message: Se implemento el parametro use_suction_cup y se resolvieron bugs del workspace - Autor: El Joho
PARAMETRO use_suction_cup (default: false): Se implemento un parametro para activar o desactivar la ventosa sin necesidad de comentar codigo manualmente. El acople (coupling_tool_end_effector_link) siempre permanece activo; solo la ventosa es opcional. Siempre existe exactamente un link end_effector activo.

Archivos modificados para el parametro use_suction_cup: - phantomx_pincher_description/urdf/phantomx_pincher_arm.xacro: parametro use_suction_cup:=false en el macro, suction_cup_link y suction_cup_joint envueltos en xacro:if, TCP del gripper en xacro:unless, TCP de la ventosa en xacro:if. - phantomx_pincher_description/urdf/phantomx_pincher.urdf.xacro: declaracion de xacro:arg use_suction_cup default=false y paso al macro. - phantomx_pincher_moveit_config/srdf/phantomx_pincher.xacro: parametro use_suction_cup en el macro SRDF, colisiones de suction_cup_link condicionadas. - phantomx_pincher_moveit_config/srdf/phantomx_pincher.srdf.xacro: declaracion del arg y paso al macro; requiere pasar name:=phantomx_pincher si se llama desde fuera de move_group.launch.py. - phantomx_pincher_moveit_config/srdf/phantomx_pincher.srdf: regenerado automaticamente. - phantomx_pincher_moveit_config/launch/move_group.launch.py: DeclareLaunchArgument use_suction_cup anadido y pasado a los comandos xacro del URDF y SRDF. - phantomx_pincher_bringup/launch/phantomx_pincher.launch.py: DeclareLaunchArgument use_suction_cup anadido, SRDF cambiado de cat a xacro con name:=phantomx_pincher y use_suction_cup, ambos IncludeLaunchDescription de move_group reciben use_suction_cup.

FIX - colcon build no actualizaba xacros en install/: CMake no trackeaba archivos .xacro como dependencias. Solucion aplicada en phantomx_pincher_description/CMakeLists.txt: stamp file con add_custom_command que depende de todos los .xacro de urdf/, forzando el install step al detectar cambios. Fix de circular dependency: target=check_xacro_files, archivo=xacro_stamp.txt. Tambien se aplico fix equivalente en phantomx_pincher_moveit_config/CMakeLists.txt para los xacros del SRDF.

FIX - move_group.launch.py standalone sin TF en RViz: joint_state_broadcaster nunca se spawneaba al lanzar move_group.launch.py directamente. Sin broadcaster no hay /joint_states y robot_state_publisher no puede calcular TF. Solucion en phantomx_pincher_moveit_config/launch/move_group.launch.py: spawner explicito de joint_state_broadcaster condicionado a IfCondition(manage_controllers) para evitar conflicto cuando se incluye desde phantomx_pincher.launch.py.

FIX - marcador interactivo de MoveIt no se actualizaba al cambiar TCP: el elemento end_effector en el SRDF tenia parent_link=suction_cup_link cuando use_suction_cup=true. MoveIt usaba ese link como objetivo IK ignorando el offset TCP del link virtual end_effector. Solucion en phantomx_pincher_moveit_config/srdf/phantomx_pincher.xacro: cambiado parent_link a end_effector en el bloque use_suction_cup=true.

DOCUMENTACION: anadido phantom_ws/src/phantomx_pincher_description/docs/ventosa_parametro_use_suction_cup.md con descripcion completa de la implementacion del parametro, archivos afectados y ejemplos de uso.

File: phantom_ws/src/phantomx_pincher_description/urdf/phantomx_pincher.urdf.xacro (robot description, xacro)
@@ -76,4 +76,8 @@
        links con joints fijos sean entidades independientes en Gazebo. -->
   <xacro:arg name="gazebo_preserve_fixed_joint" default="false"/>
+  <!-- Activa o desactiva el link y joint de la ventosa (suction cup).
+       true  → se incluye la ventosa en el modelo
+       false → solo queda el acople (coupling_tool_end_effector_link) -->
+  <xacro:arg name="use_suction_cup" default="false"/>
   <!-- ============================================================ -->
   <!-- Propiedades internas                                         -->
@@ -126,5 +130,6 @@
       ros2_control_command_interface="$(arg ros2_control_command_interface)"
       mimic_finger_joints="$(arg mimic_finger_joints)"
-      gazebo_preserve_fixed_joint="$(arg gazebo_preserve_fixed_joint)"/>
+      gazebo_preserve_fixed_joint="$(arg gazebo_preserve_fixed_joint)"
+      use_suction_cup="$(arg use_suction_cup)"/>
   <!-- ============================================================ -->
   <!-- Montaje alternativo (comentado)                              -->

File: phantom_ws/src/phantomx_pincher_description/urdf/phantomx_pincher_arm.xacro (robot description, xacro)
@@ -64,4 +64,5 @@
     mimic_finger_joints:=false
     gazebo_preserve_fixed_joint:=false
+    use_suction_cup:=false
   ">
     <!-- Link base del brazo: punto de anclaje al resto del robot -->
@@ -361,4 +362,5 @@
     </joint>
     <!-- suction cup link and joint-->
+    <xacro:if value="${use_suction_cup}">
     <link name="${prefix}suction_cup_link">
         <visual>
@@ -391,4 +393,5 @@
         <origin xyz="0 -0.01075 0.049" rpy="0 0 -${PI/2}"/>
     </joint>
+    </xacro:if>
     <!-- ====================  ${0.0115 / 2}-->
     <!-- Efector final        -->
@@ -399,25 +402,28 @@
     <!-- ==================== -->
     <!-- TCP garra, gripper   -->
-    <!-- ==================== -->
-    <!-- TCP garra, gripper-->
-    <xacro:phantomx_pincher_virtual_link
-        parent="${prefix}gripper_finger_base_link"
-        link_name="${prefix}end_effector"
-        joint_origin_xyz="${finger_centre_offset_x} 0.0 0.0"
-        joint_origin_rpy="${pi/2} ${-pi/2} ${pi/2}"
-        gazebo_preserve_fixed_joint="${gazebo_preserve_fixed_joint}"
+    <!-- Activo cuando use_suction_cup=false -->
+    <!-- ==================== -->
+    <xacro:unless value="${use_suction_cup}">
+        <xacro:phantomx_pincher_virtual_link
+            parent="${prefix}gripper_finger_base_link"
+            link_name="${prefix}end_effector"
+            joint_origin_xyz="${finger_centre_offset_x} 0.0 0.0"
+            joint_origin_rpy="${pi/2} ${-pi/2} ${pi/2}"
+            gazebo_preserve_fixed_joint="${gazebo_preserve_fixed_joint}"
+            />
+    </xacro:unless>
+    <!-- ==================== -->
+    <!-- TCP ventosa          -->
+    <!-- Activo cuando use_suction_cup=true --><!---0.114 0 -0.029-->
+    <!-- ==================== -->
+    <xacro:if value="${use_suction_cup}">
+        <xacro:phantomx_pincher_virtual_link
+            parent="${prefix}suction_cup_link"
+            link_name="${prefix}end_effector"
+            joint_origin_xyz="-0.114 0 -0.029"
+            joint_origin_rpy="0 -${PI/2} 0"
+            gazebo_preserve_fixed_joint="${gazebo_preserve_fixed_joint}"
         />
-    <!-- ==================== -->
-    <!-- TCP ventosa   -->
-    <!-- ==================== -->
-    <!-- TCP suction cop, ventosa
-    <xacro:phantomx_pincher_virtual_link
-        parent="${prefix}suction_cup_link"
-        link_name="${prefix}end_effector"
-        joint_origin_xyz="-0.114 0 -0.029"
-        joint_origin_rpy="${pi/2} ${-pi/2} ${pi/2}"
-        gazebo_preserve_fixed_joint="${gazebo_preserve_fixed_joint}"
-    />
-    -->
+    </xacro:if>
     <!-- ==================== -->
     <!-- ROS 2 Control        -->

File: phantom_ws/src/phantomx_pincher_moveit_config/srdf/phantomx_pincher.srdf.xacro (robot description, xacro)
@@ -15,7 +15,9 @@
   <!-- Prefix for all entities -->
   <xacro:arg name="use_real_gripper" default="true" />
+  <!-- Enable or disable the suction cup link and joint -->
+  <xacro:arg name="use_suction_cup" default="false" />
   <!--       -->
   <!-- Robot -->
   <!--       -->
-  <xacro:phantomx_pincher prefix="$(arg prefix)" use_real_gripper="$(arg use_real_gripper)" />
+  <xacro:phantomx_pincher prefix="$(arg prefix)" use_real_gripper="$(arg use_real_gripper)" use_suction_cup="$(arg use_suction_cup)" />
 </robot>

File: phantom_ws/src/phantomx_pincher_moveit_config/srdf/phantomx_pincher.xacro (robot description, xacro)
@@ -5,5 +5,5 @@
   <!-- Macro -->
   <!--       -->
-  <xacro:macro name="phantomx_pincher" params="prefix:=${prefix} use_real_gripper:=true">
+  <xacro:macro name="phantomx_pincher" params="prefix:=${prefix} use_real_gripper:=true use_suction_cup:=false">
     <group name="arm">
       <chain base_link="${prefix}arm_base_link" tip_link="${prefix}end_effector" />
@@ -13,6 +13,12 @@
       <joint name="${prefix}gripper_finger2_joint" />
     </group>
-    <end_effector name="${prefix}end_effector" parent_link="${prefix}gripper_finger_base_link"
-      group="gripper" parent_group="arm" />
+    <xacro:unless value="${use_suction_cup}">
+      <end_effector name="${prefix}end_effector" parent_link="${prefix}gripper_finger_base_link"
+        group="gripper" parent_group="arm" />
+    </xacro:unless>
+    <xacro:if value="${use_suction_cup}">
+      <end_effector name="${prefix}end_effector" parent_link="${prefix}end_effector"
+        group="gripper" parent_group="arm" />
+    </xacro:if>
     <virtual_joint name="${prefix}base_link_joint" type="fixed" parent_frame="world"
       child_link="${prefix}base_link" />
@@ -696,4 +702,5 @@
       <!-- C) Suction Cup SELF COLLISIONS OFF   -->
       <!-- ============================== -->
+      <xacro:if value="${use_suction_cup}">
       <!-- suction_cup_link collisions -->
       <disable_collisions link1="${prefix}suction_cup_link"
@@ -735,4 +742,5 @@
       <disable_collisions link1="${prefix}suction_cup_link"
         link2="${prefix}arm_shoulder_F3_0_link" reason="Never" />
+      </xacro:if>
     <!-- ================================================= -->
     <!-- D) ARM BASE vs KIT COLLISIONS (OFF)              -->
